File: FTDI-Toolkit-OSHW/FTDI-toolkit/FTDI-toolkit.sch (KiCad schematic (older format))
At the start: 101 parts, among them IC1 TLV70033DCKT, IC12 SN74LV1T125DCKR, IC13 74HC00BQ, IC15 TS5A3359, IC2 TLV70018DCKT, IC3 TS5A3359, IC7 SN74LV1T125DCKR, IC8 FT2232D, Y1 MQ-6.000-12-30/30/

Commit message: PCB synced with schematic, resolved all DRCs
Parts:
- removed 3V3_FT_10, 3V3_FT_11, 3V3_FT_12, 3V3_FT_13, 3V3_FT_9: 3V3_FT, symbol power:+3V3_FT
- removed 5V_USB, 5V_USB_10, 5V_USB_12, 5V_USB_13, 5V_USB_14, 5V_USB_15, 5V_USB_17, 5V_USB_18, 5V_USB_19, 5V_USB_2, 5V_USB_9: 5V_USB, symbol power:+5V_USB
- removed C1, C2, C6: 1u, symbol FTDI-toolkit-rescue:C
- removed C21, C22, C4: 100n, symbol FTDI-toolkit-rescue:C
- removed C3: 10n, symbol FTDI-toolkit-rescue:C
- removed R16, R17, R4, R5: 10k, symbol FTDI-toolkit-rescue:R
- removed R2: 470R, symbol FTDI-toolkit-rescue:R
- removed SHIELD, SHIELD_2: SHIELD, symbol power:SHIELD
- removed VCCIOA_4: VCCIOA, symbol power:VCCIOA
- removed VCCIOB_4: VCCIOB, symbol power:VCCIOB
- added C1, C2, C6: 1u, FTDI-toolkit:0603, symbol antmicroCapacitors0603:C_1u_0603
- added C21, C22, C4: C_100n_0402_16V, FTDI-toolkit:0402, symbol FTDI-toolkit-rescue:C_100n_0402_16V-antmicroCapacitors0402
- added C3: C_10n_0402, FTDI-toolkit:0402, symbol antmicroCapacitors0402:C_10n_0402
- added R16, R17, R4, R5: R_10k_0402, FTDI-toolkit:0402, symbol FTDI-toolkit-rescue:R_10k_0402-antmicroResistors0402
- added R2: R_470R_0402, FTDI-toolkit:0402, symbol antmicroResistors0402:R_470R_0402
- C5: footprint (none) -> FTDI-toolkit:0603; symbol FTDI-toolkit-rescue:C -> antmicroCapacitors0603:C_1u_0603
Connections:
- net labels added: GNDREF
- net labels removed: DIFFPAIR
- wire segments 267 -> 278
Other:
- moved on the sheet: D1, IC1, IC15, IC2, IC3, J1, L1, L2, USB1, Y1
