File: debug-toolkit.kicad_sch (KiCad schematic)
At the start: 130 parts, among them J1 USB-C_GCT_USB4105-GF-A, J1_A1 PinHeader_1x3_P2.54mm_Drill1.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, J1_B1 PinHeader_1x3_P2.54mm_Drill1.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, J2 PinHeader_2x5_P1.27mm_SMD_Shr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, J3 PinHeader_2x8_P2.54mm_Drill1mm, J4 PinHeader_1x2_P2.54mm_Drill1.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, J5 PinHeader_1x2_P1.27mm_Drill0.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, J6 PinHeader_1x4_P2.54mm_Drill1.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, J7 PinHeader_2x3_P2.54mm_Drill1.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, Q1 NX3008CBKV, Q2 NX3008CBKV, Q3 BC807-25W, Q4 SSM3K15ACT, Q5 SSM3K15ACT, Q6 SSM3K15ACT, Q7 SSM3K15ACT, U1 FT4232H_VQFN, U10 74LVC2T45_SOT833, U11 NTS0302JKZ, U12 TLV70033_SC70, U13 74HC00_DHVQFN, U14 TLV70018_SC70, U15 TS5A3359_VSSOP, U16 TS5A3359_VSSOP, U2 SN74LVC1T45_SOT-5X3, U3 SN74LVC1T45_SOT-5X3, U4 TXB0104_UQFN, U5 74LVC2T45_SOT833, U6 74LVC2T45_SOT833, U7 74LVC2T45_SOT833, U8 SN74LVC1T45_SOT-5X3, U9 SN74LVC1T45_SOT-5X3, Y1 Oscillator_12MHz_ASFLMB

Commit message: [#57618] Fix fields visibility
Parts:
- C1, C2, C36, C5, C6: Manufacturer Walsin -> KYOCERA AVX

Commit message: [#57618] Fix diodes polarization
Connections:
- net 3V3_FT: now also D3.1 (C); no longer D3.2 (A)
- net 5V_USB: now also 1V8_A1.2 (A), 1V8_B1.2 (A), 3V3_A1.2 (A), 3V3_B1.2 (A), 5V0_A1.2 (A), 5V0_B1.2 (A), USB1.2 (A); no longer 1V8_A1.1 (C), 1V8_B1.1 (C), 3V3_A1.1 (C), 3V3_B1.1 (C), 5V0_A1.1 (C), 5V0_B1.1 (C), USB1.1 (C)
- net GND: now also RX_A1.1 (C), RX_B1.1 (C), TX_A1.1 (C), TX_B1.1 (C); no longer RX_A1.2 (A), RX_B1.2 (A), TX_A1.2 (A), TX_B1.2 (A)
- net SDA: now also D4.2 (A); no longer D4.1 (C)
- net at R2.2: now also USB1.1 (C); no longer USB1.2 (A)
- net at C33.2, R34.1, U11.1 (VCC_A): now also D3.2 (A); no longer D3.1 (C)
- net at Q4.3 (D), R11.1: now also TX_B1.2 (A); no longer TX_A1.1 (C)
- net at Q6.3 (D), R12.1: now also RX_B1.2 (A); no longer RX_A1.1 (C)
- net at Q5.3 (D), R14.1: now also TX_A1.2 (A); no longer TX_B1.1 (C)
- net at Q7.3 (D), R15.1: now also RX_A1.2 (A); no longer RX_B1.1 (C)
- net at R1.1: now also 3V3_A1.1 (C); no longer 3V3_A1.2 (A)
- net at R3.1: now also 1V8_A1.1 (C); no longer 1V8_A1.2 (A)
- net at R6.1: now also 5V0_A1.1 (C); no longer 5V0_A1.2 (A)
- net at R7.1: now also 3V3_B1.1 (C); no longer 3V3_B1.2 (A)
- net at R8.1: now also 1V8_B1.1 (C); no longer 1V8_B1.2 (A)
- net at R18.1: now also 5V0_B1.1 (C); no longer 5V0_B1.2 (A)
- net at U7.7 (1B): now also D4.1 (C); no longer D4.2 (A)
Other:
- moved on the sheet: D3, D4, RX_A1, RX_B1, TX_A1, TX_B1, U13, USB1
