File: debug-toolkit.kicad_sch (KiCad schematic)
At the start: 130 parts, among them J1 USB-C_GCT_USB4105-GF-A, J1_A1 PinHeader_1x3_P2.54mm_Drill1.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, J1_B1 PinHeader_1x3_P2.54mm_Drill1.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, J2 PinHeader_2x5_P1.27mm_SMD_Shr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, J3 PinHeader_2x8_P2.54mm_Drill1mm, J4 PinHeader_1x2_P2.54mm_Drill1.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, J5 PinHeader_1x2_P1.27mm_Drill0.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, J6 PinHeader_1x4_P2.54mm_Drill1.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, J7 PinHeader_2x3_P2.54mm_Drill1.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, Q1 NX3008CBKV, Q2 NX3008CBKV, Q3 BC807-25W, Q4 SSM3K15ACT, Q5 SSM3K15ACT, Q6 SSM3K15ACT, Q7 SSM3K15ACT, U1 FT4232H_VQFN, U10 74LVC2T45_SOT833, U11 NTS0302JKZ, U12 TLV70033_SC70, U13 74HC00_DHVQFN, U14 TLV70018_SC70, U15 TS5A3359_VSSOP, U16 TS5A3359_VSSOP, U2 SN74LVC1T45_SOT-5X3, U3 SN74LVC1T45_SOT-5X3, U4 TXB0104_UQFN, U5 74LVC2T45_SOT833, U6 74LVC2T45_SOT833, U7 74LVC2T45_SOT833, U8 SN74LVC1T45_SOT-5X3, U9 SN74LVC1T45_SOT-5X3, Y1 Oscillator_12MHz_ASFLMB

Commit message: [#57618] Fix ERC
Parts:
- 1V8_A1, 1V8_B1, 3V3_A1, 3V3_B1, 5V0_A1, 5V0_B1, C1, C11, C2, C23, C27, C3, C33, C36, C5, C6, D3, D4, FB1, FB2, L1, L2, N1, N2, R1, R10, R11, R12, R13, R14, R15, R16, R17, R18, R19, R2, R20, R21, R22, R23, R24, R25, R26, R27, R28, R29, R3, R30, R31, R32, R33, R34, R35, R36, R37, R38, R39, R4, R40, R5, R6, R7, R8, R9, RX_A1, RX_B1, TX_A1, TX_B1, USB1, Y1: Public (none) -> False
Other:
- moved on the sheet: C15, C16, C24, C26, C27, C28, C29, FB1, Q4, R10, R27, R4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
